File: EEG_v2_micro.sch (KiCad schematic (older format))
At the start: 34 parts, among them SW3 SW_PUSH, SW4 SW_PUSH, U6 CC2540, U7 2450BM15A0002E, X1 32-KHz, X2 32-MHz

Commit message: Associate footprints to pcbnew
Parts:
- removed C51: 100n, 0402_X5R_K_10, symbol C
- C43: value 2.2u -> 1u; footprint 0402_X5R_M_6P3VDC -> 0402_X5R_K_6P3
- C44, C47, C48, C50: value 100n -> 1u; footprint 0402_X5R_K_10 -> 0402_X5R_K_6P3
- C45: value 10p -> 1u; footprint 0402_NP0_J_50 -> 0402_X5R_K_6P3
- C49: value 220p -> 1u; footprint 0402_NP0_J_50 -> 0402_X5R_K_6P3
- renumbered C52 to C51, C53 to C52, C54 to C53, C55 to C54, C56 to C55, C57 to C56, C58 to C57, C59 to C58, C60 to C59
Changed lines of the file:
@@
 $EndComp
 $Comp
-L C C54
+L C C53
 U 1 1 54B4DAF5
 P 3400 3550
-F 0 "C54" H 3400 3650 40  0000 L CNN
+F 0 "C53" H 3400 3650 40  0000 L CNN
 F 1 "1u" H 3406 3465 40  0000 L CNN
 F 2 "0402_X5R_K_6P3" H 3438 3400 30  0000 C CNN
@@
 $EndComp
 $Comp
-L C C58
+L C C57
 U 1 1 54B4E0D9
 P 5750 6250
-F 0 "C58" H 5750 6350 40  0000 L CNN
+F 0 "C57" H 5750 6350 40  0000 L CNN
 F 1 "12p" H 5756 6165 40  0000 L CNN
 F 2 "0402_NP0_J_50" H 5788 6100 30  0000 C CNN
@@
 $EndComp
 $Comp
-L C C59
+L C C58
 U 1 1 54B4E0DF
 P 6350 6250
-F 0 "C59" H 6350 6350 40  0000 L CNN
+F 0 "C58" H 6350 6350 40  0000 L CNN
 F 1 "12p" H 6356 6165 40  0000 L CNN
 F 2 "0402_NP0_J_50" H 6388 6100 30  0000 C CNN
@@
 $EndComp
 $Comp
-L C C53
+L C C52
 U 1 1 54B4E361
 P 4950 2500
-F 0 "C53" H 4950 2600 40  0000 L CNN
+F 0 "C52" H 4950 2600 40  0000 L CNN
 F 1 "15p" H 4956 2415 40  0000 L CNN
 F 2 "0402_NP0_J_50" H 4988 2350 30  0000 C CNN
@@
 $EndComp
 $Comp
-L C C52
+L C C51
 U 1 1 54B4E367
 P 4350 2500
-F 0 "C52" H 4350 2600 40  0000 L CNN
+F 0 "C51" H 4350 2600 40  0000 L CNN
 F 1 "15p" H 4356 2415 40  0000 L CNN
 F 2 "0402_NP0_J_50" H 4388 2350 30  0000 C CNN
@@
 SCK
 $Comp
-L C C44
-U 1 1 54B6FDC9
-P 2350 1700
-F 0 "C44" H 2350 1800 40  0000 L CNN
-F 1 "100n" H 2356 1615 40  0000 L CNN
-F 2 "0402_X5R_K_10" H 2388 1550 30  0000 C CNN
-F 3 "~" H 2350 1700 60  0000 C CNN
-	1    2350 1700
-	1    0    0    -1
-$EndComp
-$Comp
-L C C43
-U 1 1 54B6FDD8
-P 1700 1700
-F 0 "C43" H 1700 1800 40  0000 L CNN
-F 1 "2.2u" H 1706 1615 40  0000 L CNN
-F 2 "0402_X5R_M_6P3VDC" H 1738 1550 30  0000 C CNN
-F 3 "~" H 1700 1700 60  0000 C CNN
-	1    1700 1700
-	1    0    0    -1
-$EndComp
-$Comp
 L INDUCTOR L1
 U 1 1 54B6FE82
@@
 $EndComp
 $Comp
-L C C47
-U 1 1 54B708C7
-P 5400 1750
-F 0 "C47" H 5400 1850 40  0000 L CNN
-F 1 "100n" H 5406 1665 40  0000 L CNN
-F 2 "0402_X5R_K_10" H 5438 1600 30  0000 C CNN
-F 3 "~" H 5400 1750 60  0000 C CNN
-	1    5400 1750
-	1    0    0    -1
-$EndComp
-$Comp
 L AGND #PWR053
 U 1 1 54B708CD
@@
 $EndComp
 $Comp
-L C C48
-U 1 1 54B70B01
-P 5950 1750
-F 0 "C48" H 5950 1850 40  0000 L CNN
-F 1 "100n" H 5956 1665 40  0000 L CNN
-F 2 "0402_X5R_K_10" H 5988 1600 30  0000 C CNN
-F 3 "~" H 5950 1750 60  0000 C CNN
-	1    5950 1750
-	1    0    0    -1
-$EndComp
-$Comp
 L AGND #PWR054
 U 1 1 54B70B07
@@
 $EndComp
 $Comp
-L C C49
-U 1 1 54B70B0E
-P 6350 1750
-F 0 "C49" H 6350 1850 40  0000 L CNN
-F 1 "220p" H 6356 1665 40  0000 L CNN
-F 2 "0402_NP0_J_50" H 6388 1600 30  0000 C CNN
-F 3 "~" H 6350 1750 60  0000 C CNN
-	1    6350 1750
-	1    0    0    -1
-$EndComp
-$Comp
 L AGND #PWR055
-U 1 1 54B70B14
-P 6350 2050
-F 0 "#PWR055" H 6350 2050 40  0001 C CNN
-F 1 "AGND" H 6350 1980 50  0000 C CNN
-F 2 "~" H 6350 2050 60  0000 C CNN
-F 3 "~" H 6350 2050 60  0000 C CNN
-	1    6350 2050
-	1    0    0    -1
-$EndComp
-$Comp
-L C C50
-U 1 1 54B70FFF
-P 6950 1750
-F 0 "C50" H 6950 1850 40  0000 L CNN
-F 1 "100n" H 6956 1665 40  0000 L CNN
-F 2 "0402_X5R_K_10" H 6988 1600 30  0000 C CNN
-F 3 "~" H 6950 1750 60  0000 C CNN
-	1    6950 1750
-	1    0    0    -1
-$EndComp
-$Comp
-L AGND #PWR056
 U 1 1 54B71005
 P 6950 2050
-F 0 "#PWR056" H 6950 2050 40  0001 C CNN
+F 0 "#PWR055" H 6950 2050 40  0001 C CNN
 F 1 "AGND" H 6950 1980 50  0000 C CNN
 F 2 "~" H 6950 2050 60  0000 C CNN
@@
 $EndComp
 $Comp
-L C C51
-U 1 1 54B7105B
-P 7500 1750
-F 0 "C51" H 7500 1850 40  0000 L CNN
-F 1 "100n" H 7506 1665 40  0000 L CNN
-F 2 "0402_X5R_K_10" H 7538 1600 30  0000 C CNN
-F 3 "~" H 7500 1750 60  0000 C CNN
-	1    7500 1750
-	1    0    0    -1
-$EndComp
-$Comp
-L AGND #PWR057
+L AGND #PWR056
 U 1 1 54B71061
 P 7500 2050
-F 0 "#PWR057" H 7500 2050 40  0001 C CNN
+F 0 "#PWR056" H 7500 2050 40  0001 C CNN
 F 1 "AGND" H 7500 1980 50  0000 C CNN
 F 2 "~" H 7500 2050 60  0000 C CNN
@@
 $EndComp
 $Comp
-L AGND #PWR058
+L AGND #PWR057
 U 1 1 54B71D5A
 P 8450 5400
-F 0 "#PWR058" H 8450 5400 40  0001 C CNN
+F 0 "#PWR057" H 8450 5400 40  0001 C CNN
 F 1 "AGND" H 8450 5330 50  0000 C CNN
 F 2 "~" H 8450 5400 60  0000 C CNN
@@
 Wire Wire Line
 	5950 1950 5950 2050
-Wire Wire Line
-	6350 1950 6350 2050
-Wire Wire Line
-	5700 1550 6350 1550
-Connection ~ 5950 1550
 Connection ~ 5700 1550
 Wire Wire Line
@@
 RESET_ADS
 $Comp
-L C C45
-U 1 1 54B75300
-P 3050 1700
-F 0 "C45" H 3050 1800 40  0000 L CNN
-F 1 "10p" H 3056 1615 40  0000 L CNN
-F 2 "0402_NP0_J_50" H 3088 1550 30  0000 C CNN
-F 3 "~" H 3050 1700 60  0000 C CNN
-	1    3050 1700
-	1    0    0    -1
-$EndComp
-$Comp
-L AGND #PWR059
+L AGND #PWR058
 U 1 1 54B75306
 P 3050 2000
-F 0 "#PWR059" H 3050 2000 40  0001 C CNN
+F 0 "#PWR058" H 3050 2000 40  0001 C CNN
 F 1 "AGND" H 3050 1930 50  0000 C CNN
 F 2 "~" H 3050 2000 60  0000 C CNN
@@
 	1050 4650 900  4650
 $Comp
-L C C56
+L C C55
 U 1 1 54B75968
 P 1800 4800
-F 0 "C56" H 1800 4900 40  0000 L CNN
+F 0 "C55" H 1800 4900 40  0000 L CNN
 F 1 "47p" H 1806 4715 40  0000 L CNN
 F 2 "0402_NP0_J_50" H 1838 4650 30  0000 C CNN
@@
 $EndComp
 $Comp
-L C C55
+L C C54
 U 1 1 54B75989
 P 1800 4300
-F 0 "C55" H 1800 4400 40  0000 L CNN
+F 0 "C54" H 1800 4400 40  0000 L CNN
 F 1 "47p" H 1806 4215 40  0000 L CNN
 F 2 "0402_NP0_J_50" H 1838 4150 30  0000 C CNN
@@
 $EndComp
 $Comp
-L AGND #PWR060
+L AGND #PWR059
 U 1 1 54B75999
 P 1800 5050
-F 0 "#PWR060" H 1800 5050 40  0001 C CNN
+F 0 "#PWR059" H 1800 5050 40  0001 C CNN
 F 1 "AGND" H 1800 4980 50  0000 C CNN
 F 2 "~" H 1800 5050 60  0000 C CNN
@@
 $EndComp
 $Comp
-L AGND #PWR061
+L AGND #PWR060
 U 1 1 54B7599F
 P 1800 4000
-F 0 "#PWR061" H 1800 4000 40  0001 C CNN
+F 0 "#PWR060" H 1800 4000 40  0001 C CNN
 F 1 "AGND" H 1800 3930 50  0000 C CNN
 F 2 "~" H 1800 4000 60  0000 C CNN
@@
 NoConn ~ 4100 6000
 $Comp
-L C C60
+L C C59
 U 1 1 54C2E982
 P 4600 7350
-F 0 "C60" H 4600 7450 40  0000 L CNN
+F 0 "C59" H 4600 7450 40  0000 L CNN
 F 1 "1n" H 4606 7265 40  0000 L CNN
 F 2 "0402_NP0_J_50" H 4638 7200 30  0000 C CNN
@@
 	4600 6000 4600 7150
 $Comp
-L AGND #PWR062
+L AGND #PWR061
 U 1 1 54C2E9F6
 P 4600 7600
-F 0 "#PWR062" H 4600 7600 40  0001 C CNN
+F 0 "#PWR061" H 4600 7600 40  0001 C CNN
 F 1 "AGND" H 4600 7530 50  0000 C CNN
 F 2 "~" H 4600 7600 60  0000 C CNN
@@
 	5250 7150 5400 7150
 $Comp
-L C C57
+L C C56
 U 1 1 54C2ECFD
 P 9900 5150
-F 0 "C57" H 9900 5250 40  0000 L CNN
+F 0 "C56" H 9900 5250 40  0000 L CNN
 F 1 "0.5p" H 9906 5065 40  0000 L CNN
 F 2 "0402_NP0_B_50" H 9938 5000 30  0000 C CNN
@@
 $EndComp
 $Comp
-L AGND #PWR063
+L AGND #PWR062
 U 1 1 54C2ED03
 P 9900 5550
-F 0 "#PWR063" H 9900 5550 40  0001 C CNN
+F 0 "#PWR062" H 9900 5550 40  0001 C CNN
 F 1 "AGND" H 9900 5480 50  0000 C CNN
 F 2 "~" H 9900 5550 60  0000 C CNN
@@
 $EndComp
 $Comp
-L AGND #PWR064
+L AGND #PWR063
 U 1 1 54C2EF06
 P 9450 4200
-F 0 "#PWR064" H 9450 4200 40  0001 C CNN
+F 0 "#PWR063" H 9450 4200 40  0001 C CNN
 F 1 "AGND" H 9450 4130 50  0000 C CNN
 F 2 "~" H 9450 4200 60  0000 C CNN
@@
 	2300 6100 2300 6350
 $Comp
-L AGND #PWR065
+L AGND #PWR064
 U 1 1 54CBF6E0
 P 2300 6350
-F 0 "#PWR065" H 2300 6350 40  0001 C CNN
+F 0 "#PWR064" H 2300 6350 40  0001 C CNN
 F 1 "AGND" H 2300 6280 50  0000 C CNN
 F 2 "~" H 2300 6350 60  0000 C CNN
@@
 	2600 6100 2600 6350
 $Comp
-L AGND #PWR066
+L AGND #PWR065
 U 1 1 54CBFC8B
 P 2600 6350
-F 0 "#PWR066" H 2600 6350 40  0001 C CNN
+F 0 "#PWR065" H 2600 6350 40  0001 C CNN
 F 1 "AGND" H 2600 6280 50  0000 C CNN
 F 2 "~" H 2600 6350 60  0000 C CNN
@@
 	2900 6950 2900 6900
 $Comp
-L AGND #PWR067
+L AGND #PWR066
 U 1 1 54CC0292
 P 3150 7450
-F 0 "#PWR067" H 3150 7450 40  0001 C CNN
+F 0 "#PWR066" H 3150 7450 40  0001 C CNN
 F 1 "AGND" H 3150 7380 50  0000 C CNN
 F 2 "~" H 3150 7450 60  0000 C CNN
@@
 $EndComp
 $Comp
-L AGND #PWR068
+L AGND #PWR067
 U 1 1 54CC0298
 P 2900 7450
-F 0 "#PWR068" H 2900 7450 40  0001 C CNN
+F 0 "#PWR067" H 2900 7450 40  0001 C CNN
 F 1 "AGND" H 2900 7380 50  0000 C CNN
 F 2 "~" H 2900 7450 60  0000 C CNN
@@
 NoConn ~ 3000 4800
 NoConn ~ 3000 4900
+$Comp
+L C C45
+U 1 1 54D07EA2
+P 3050 1700
+F 0 "C45" H 3050 1800 40  0000 L CNN
+F 1 "1u" H 3056 1615 40  0000 L CNN
+F 2 "0402_X5R_K_6P3" H 3088 1550 30  0000 C CNN
+F 3 "~" H 3050 1700 60  0000 C CNN
+	1    3050 1700
+	1    0    0    -1
+$EndComp
+$Comp
+L C C44
+U 1 1 54D07EA8
+P 2350 1700
+F 0 "C44" H 2350 1800 40  0000 L CNN
+F 1 "1u" H 2356 1615 40  0000 L CNN
+F 2 "0402_X5R_K_6P3" H 2388 1550 30  0000 C CNN
+F 3 "~" H 2350 1700 60  0000 C CNN
+	1    2350 1700
+	1    0    0    -1
+$EndComp
+$Comp
+L C C47
+U 1 1 54D07EAE
+P 5400 1750
+F 0 "C47" H 5400 1850 40  0000 L CNN
+F 1 "1u" H 5406 1665 40  0000 L CNN
+F 2 "0402_X5R_K_6P3" H 5438 1600 30  0000 C CNN
+F 3 "~" H 5400 1750 60  0000 C CNN
+	1    5400 1750
+	1    0    0    -1
+$EndComp
+$Comp
+L C C48
+U 1 1 54D07EB4
+P 5950 1750
+F 0 "C48" H 5950 1850 40  0000 L CNN
+F 1 "1u" H 5956 1665 40  0000 L CNN
+F 2 "0402_X5R_K_6P3" H 5988 1600 30  0000 C CNN
+F 3 "~" H 5950 1750 60  0000 C CNN
+	1    5950 1750
+	1    0    0    -1
+$EndComp
+Wire Wire Line
+	5950 1550 5700 1550
+$Comp
+L C C43
+U 1 1 54D07F4C
+P 1700 1700
+F 0 "C43" H 1700 1800 40  0000 L CNN
+F 1 "1u" H 1706 1615 40  0000 L CNN
+F 2 "0402_X5R_K_6P3" H 1738 1550 30  0000 C CNN
+F 3 "~" H 1700 1700 60  0000 C CNN
+	1    1700 1700
+	1    0    0    -1
+$EndComp
+$Comp
+L C C49
+U 1 1 54D07F52
+P 6950 1750
+F 0 "C49" H 6950 1850 40  0000 L CNN
+F 1 "1u" H 6956 1665 40  0000 L CNN
+F 2 "0402_X5R_K_6P3" H 6988 1600 30  0000 C CNN
+F 3 "~" H 6950 1750 60  0000 C CNN
+	1    6950 1750
+	1    0    0    -1
+$EndComp
+$Comp
+L C C50
+U 1 1 54D07F58
+P 7500 1750
+F 0 "C50" H 7500 1850 40  0000 L CNN
+F 1 "1u" H 7506 1665 40  0000 L CNN
+F 2 "0402_X5R_K_6P3" H 7538 1600 30  0000 C CNN
+F 3 "~" H 7500 1750 60  0000 C CNN
+	1    7500 1750
+	1    0    0    -1
+$EndComp
 $EndSCHEMATC

Commit message: Begin layout. Finish footprints and association.
Parts:
- removed X1: 32-KHz, ~, symbol QUARTZCMS4
- added X1: QUARTZCMS4_32K, ~, symbol QUARTZCMS4_32K
Changed lines of the file:
@@
 Sheet 4 4
 Title "Project Synapse Prototype Board"
-Date "29 jan 2015"
+Date "31 jan 2015"
 Rev "A.b"
 Comp "Senior Design 14-15"
@@
 $EndComp
 $Comp
-L QUARTZCMS4 X1
-U 1 1 54B4E2E4
-P 4650 3000
-F 0 "X1" H 4650 3150 60  0000 C CNN
-F 1 "32-KHz" H 4650 2850 60  0000 C CNN
-F 2 "~" H 4650 3000 60  0000 C CNN
-F 3 "~" H 4650 3000 60  0000 C CNN
-	1    4650 3000
-	-1   0    0    1
-$EndComp
-$Comp
 L C C52
 U 1 1 54B4E361
@@
 	1    0    0    -1
 $EndComp
+$Comp
+L QUARTZCMS4_32K X1
+U 1 1 54CD5E89
+P 4650 3000
+F 0 "X1" H 4650 3150 60  0000 C CNN
+F 1 "QUARTZCMS4_32K" H 4650 2850 60  0000 C CNN
+F 2 "~" H 4650 3000 60  0000 C CNN
+F 3 "~" H 4650 3000 60  0000 C CNN
+	1    4650 3000
+	1    0    0    -1
+$EndComp
