File: EEG_v2_micro.sch (KiCad schematic (older format))
At the start: 33 parts, among them SW3 SW_PUSH, SW4 SW_PUSH, U6 CC2540, U7 2450BM15A0002E, X1 QUARTZCMS4_32K, X2 32-MHz

Commit message: Change USB connector. Continue layout.
Parts:
- removed SW3, SW4: SW_PUSH, Thru 1825910, symbol SW_PUSH
- added SW3, SW4: SW_PUSH_4PIN, ~, symbol SW_PUSH_4PIN
Connections:
- wire segments 110 -> 118
Changed lines of the file:
@@
 Sheet 4 4
 Title "Project Synapse Prototype Board"
-Date "31 jan 2015"
+Date "1 feb 2015"
 Rev "A.b"
 Comp "Senior Design 14-15"
@@
 $EndComp
 $Comp
-L AGND #PWR041
+L AGND #PWR040
 U 1 1 54B4DC2F
 P 3400 3850
-F 0 "#PWR041" H 3400 3850 40  0001 C CNN
+F 0 "#PWR040" H 3400 3850 40  0001 C CNN
 F 1 "AGND" H 3400 3780 50  0000 C CNN
 F 2 "~" H 3400 3850 60  0000 C CNN
@@
 $EndComp
 $Comp
-L AGND #PWR042
+L AGND #PWR041
 U 1 1 54B4DEBC
 P 6550 4450
-F 0 "#PWR042" H 6550 4450 40  0001 C CNN
+F 0 "#PWR041" H 6550 4450 40  0001 C CNN
 F 1 "AGND" H 6550 4380 50  0000 C CNN
 F 2 "~" H 6550 4450 60  0000 C CNN
@@
 $EndComp
 $Comp
-L +3.3V #PWR043
+L +3.3V #PWR042
 U 1 1 54B4DF64
 P 650 1400
-F 0 "#PWR043" H 650 1360 30  0001 C CNN
+F 0 "#PWR042" H 650 1360 30  0001 C CNN
 F 1 "+3.3V" H 650 1510 30  0000 C CNN
 F 2 "~" H 650 1400 60  0000 C CNN
@@
 $EndComp
 $Comp
-L AGND #PWR044
+L AGND #PWR043
 U 1 1 54B4E155
 P 5750 6600
-F 0 "#PWR044" H 5750 6600 40  0001 C CNN
+F 0 "#PWR043" H 5750 6600 40  0001 C CNN
 F 1 "AGND" H 5750 6530 50  0000 C CNN
 F 2 "~" H 5750 6600 60  0000 C CNN
@@
 $EndComp
 $Comp
-L AGND #PWR045
+L AGND #PWR044
 U 1 1 54B4E15B
 P 6350 6600
-F 0 "#PWR045" H 6350 6600 40  0001 C CNN
+F 0 "#PWR044" H 6350 6600 40  0001 C CNN
 F 1 "AGND" H 6350 6530 50  0000 C CNN
 F 2 "~" H 6350 6600 60  0000 C CNN
@@
 $EndComp
 $Comp
-L AGND #PWR046
+L AGND #PWR045
 U 1 1 54B4E36D
 P 4950 2150
-F 0 "#PWR046" H 4950 2150 40  0001 C CNN
+F 0 "#PWR045" H 4950 2150 40  0001 C CNN
 F 1 "AGND" H 4950 2080 50  0000 C CNN
 F 2 "~" H 4950 2150 60  0000 C CNN
@@
 $EndComp
 $Comp
-L AGND #PWR047
+L AGND #PWR046
 U 1 1 54B4E373
 P 4350 2150
-F 0 "#PWR047" H 4350 2150 40  0001 C CNN
+F 0 "#PWR046" H 4350 2150 40  0001 C CNN
 F 1 "AGND" H 4350 2080 50  0000 C CNN
 F 2 "~" H 4350 2150 60  0000 C CNN
@@
 $EndComp
 $Comp
-L AGND #PWR048
+L AGND #PWR047
 U 1 1 54B4E516
 P 4400 5300
-F 0 "#PWR048" H 4400 5300 40  0001 C CNN
+F 0 "#PWR047" H 4400 5300 40  0001 C CNN
 F 1 "AGND" H 4400 5230 50  0000 C CNN
 F 2 "~" H 4400 5300 60  0000 C CNN
@@
 $EndComp
 $Comp
-L AGND #PWR049
+L AGND #PWR048
 U 1 1 54B4E69D
 P 2500 4250
-F 0 "#PWR049" H 2500 4250 40  0001 C CNN
+F 0 "#PWR048" H 2500 4250 40  0001 C CNN
 F 1 "AGND" H 2500 4180 50  0000 C CNN
 F 2 "~" H 2500 4250 60  0000 C CNN
@@
 	-1   0    0    1
 $EndComp
+Text HLabel 4100 6200 3    60   Output ~ 0
+MOSI
+Text HLabel 4000 6200 3    60   Input ~ 0
+MISO
 Text HLabel 4200 6200 3    60   Output ~ 0
-MOSI
-Text HLabel 4300 6200 3    60   Input ~ 0
-MISO
-Text HLabel 4000 6200 3    60   Output ~ 0
 SCK
 $Comp
@@
 $EndComp
 $Comp
-L AGND #PWR050
+L AGND #PWR049
 U 1 1 54B6FF14
 P 2350 2000
-F 0 "#PWR050" H 2350 2000 40  0001 C CNN
+F 0 "#PWR049" H 2350 2000 40  0001 C CNN
 F 1 "AGND" H 2350 1930 50  0000 C CNN
 F 2 "~" H 2350 2000 60  0000 C CNN
@@
 $EndComp
 $Comp
-L AGND #PWR051
+L AGND #PWR050
 U 1 1 54B7020B
 P 1700 2000
-F 0 "#PWR051" H 1700 2000 40  0001 C CNN
+F 0 "#PWR050" H 1700 2000 40  0001 C CNN
 F 1 "AGND" H 1700 1930 50  0000 C CNN
 F 2 "~" H 1700 2000 60  0000 C CNN
@@
 $EndComp
 $Comp
-L AGND #PWR052
+L AGND #PWR051
 U 1 1 54B703A3
 P 3600 2000
-F 0 "#PWR052" H 3600 2000 40  0001 C CNN
+F 0 "#PWR051" H 3600 2000 40  0001 C CNN
 F 1 "AGND" H 3600 1930 50  0000 C CNN
 F 2 "~" H 3600 2000 60  0000 C CNN
@@
 $EndComp
 $Comp
-L AGND #PWR053
+L AGND #PWR052
 U 1 1 54B708CD
 P 5400 2050
-F 0 "#PWR053" H 5400 2050 40  0001 C CNN
+F 0 "#PWR052" H 5400 2050 40  0001 C CNN
 F 1 "AGND" H 5400 1980 50  0000 C CNN
 F 2 "~" H 5400 2050 60  0000 C CNN
@@
 $EndComp
 $Comp
-L AGND #PWR054
+L AGND #PWR053
 U 1 1 54B70B07
 P 5950 2050
-F 0 "#PWR054" H 5950 2050 40  0001 C CNN
+F 0 "#PWR053" H 5950 2050 40  0001 C CNN
 F 1 "AGND" H 5950 1980 50  0000 C CNN
 F 2 "~" H 5950 2050 60  0000 C CNN
@@
 $EndComp
 $Comp
-L AGND #PWR055
+L AGND #PWR054
 U 1 1 54B71005
 P 6950 2050
-F 0 "#PWR055" H 6950 2050 40  0001 C CNN
+F 0 "#PWR054" H 6950 2050 40  0001 C CNN
 F 1 "AGND" H 6950 1980 50  0000 C CNN
 F 2 "~" H 6950 2050 60  0000 C CNN
@@
 $EndComp
 $Comp
-L AGND #PWR056
+L AGND #PWR055
 U 1 1 54B71061
 P 7500 2050
-F 0 "#PWR056" H 7500 2050 40  0001 C CNN
+F 0 "#PWR055" H 7500 2050 40  0001 C CNN
 F 1 "AGND" H 7500 1980 50  0000 C CNN
 F 2 "~" H 7500 2050 60  0000 C CNN
@@
 $EndComp
 $Comp
-L AGND #PWR057
+L AGND #PWR056
 U 1 1 54B71D5A
 P 8450 5400
-F 0 "#PWR057" H 8450 5400 40  0001 C CNN
+F 0 "#PWR056" H 8450 5400 40  0001 C CNN
 F 1 "AGND" H 8450 5330 50  0000 C CNN
 F 2 "~" H 8450 5400 60  0000 C CNN
@@
 	4200 6000 4200 6200
 Wire Wire Line
-	4300 6000 4300 6200
-Wire Wire Line
 	3400 3750 3400 3850
 Wire Wire Line
@@
 Wire Wire Line
 	9900 4600 9900 4950
-Text HLabel 4400 6200 3    60   Input ~ 0
+Text HLabel 3900 6200 3    60   Input ~ 0
 DRDY
 Text HLabel 4500 6200 3    60   Output ~ 0
 START
-Text HLabel 3900 6200 3    60   Output ~ 0
+Text HLabel 4400 6200 3    60   Output ~ 0
 CS
 Text HLabel 3800 6200 3    60   Output ~ 0
 RESET_ADS
 $Comp
-L AGND #PWR058
+L AGND #PWR057
 U 1 1 54B75306
 P 3050 2000
-F 0 "#PWR058" H 3050 2000 40  0001 C CNN
+F 0 "#PWR057" H 3050 2000 40  0001 C CNN
 F 1 "AGND" H 3050 1930 50  0000 C CNN
 F 2 "~" H 3050 2000 60  0000 C CNN
@@
 $EndComp
 $Comp
-L AGND #PWR059
+L AGND #PWR058
 U 1 1 54B75999
 P 1800 5050
-F 0 "#PWR059" H 1800 5050 40  0001 C CNN
+F 0 "#PWR058" H 1800 5050 40  0001 C CNN
 F 1 "AGND" H 1800 4980 50  0000 C CNN
 F 2 "~" H 1800 5050 60  0000 C CNN
@@
 $EndComp
 $Comp
-L AGND #PWR060
+L AGND #PWR059
 U 1 1 54B7599F
 P 1800 4000
-F 0 "#PWR060" H 1800 4000 40  0001 C CNN
+F 0 "#PWR059" H 1800 4000 40  0001 C CNN
 F 1 "AGND" H 1800 3930 50  0000 C CNN
 F 2 "~" H 1800 4000 60  0000 C CNN
@@
 Wire Wire Line
 	3800 6000 3800 6200
-NoConn ~ 4100 6000
 $Comp
 L C C59
@@
 	4600 6000 4600 7150
 $Comp
-L AGND #PWR061
+L AGND #PWR060
 U 1 1 54C2E9F6
 P 4600 7600
-F 0 "#PWR061" H 4600 7600 40  0001 C CNN
+F 0 "#PWR060" H 4600 7600 40  0001 C CNN
 F 1 "AGND" H 4600 7530 50  0000 C CNN
 F 2 "~" H 4600 7600 60  0000 C CNN
@@
 $EndComp
 $Comp
-L AGND #PWR062
+L AGND #PWR061
 U 1 1 54C2ED03
 P 9900 5550
-F 0 "#PWR062" H 9900 5550 40  0001 C CNN
+F 0 "#PWR061" H 9900 5550 40  0001 C CNN
 F 1 "AGND" H 9900 5480 50  0000 C CNN
 F 2 "~" H 9900 5550 60  0000 C CNN
@@
 $EndComp
 $Comp
-L AGND #PWR063
+L AGND #PWR062
 U 1 1 54C2EF06
 P 9450 4200
-F 0 "#PWR063" H 9450 4200 40  0001 C CNN
+F 0 "#PWR062" H 9450 4200 40  0001 C CNN
 F 1 "AGND" H 9450 4130 50  0000 C CNN
 F 2 "~" H 9450 4200 60  0000 C CNN
@@
 Wire Wire Line
 	3750 3350 3400 3350
-$Comp
-L SW_PUSH SW3
-U 1 1 54CBF5D1
-P 2300 5800
-F 0 "SW3" H 2450 5910 50  0000 C CNN
-F 1 "SW_PUSH" H 2300 5720 50  0000 C CNN
-F 2 "Thru 1825910" H 2300 5800 60  0001 C CNN
-F 3 "~" H 2300 5800 60  0000 C CNN
-	1    2300 5800
-	0    -1   -1   0
-$EndComp
 Wire Wire Line
 	2300 6100 2300 6350
 $Comp
-L AGND #PWR064
+L AGND #PWR063
 U 1 1 54CBF6E0
 P 2300 6350
-F 0 "#PWR064" H 2300 6350 40  0001 C CNN
+F 0 "#PWR063" H 2300 6350 40  0001 C CNN
 F 1 "AGND" H 2300 6280 50  0000 C CNN
 F 2 "~" H 2300 6350 60  0000 C CNN
@@
 Wire Wire Line
 	3150 6200 3700 6200
-$Comp
-L SW_PUSH SW4
-U 1 1 54CBFC84
-P 2600 5800
-F 0 "SW4" H 2750 5910 50  0000 C CNN
-F 1 "SW_PUSH" H 2600 5720 50  0000 C CNN
-F 2 "Thru 1825910" H 2600 5800 60  0001 C CNN
-F 3 "~" H 2600 5800 60  0000 C CNN
-	1    2600 5800
-	0    -1   -1   0
-$EndComp
 Wire Wire Line
 	2600 6100 2600 6350
 $Comp
-L AGND #PWR065
+L AGND #PWR064
 U 1 1 54CBFC8B
 P 2600 6350
-F 0 "#PWR065" H 2600 6350 40  0001 C CNN
+F 0 "#PWR064" H 2600 6350 40  0001 C CNN
 F 1 "AGND" H 2600 6280 50  0000 C CNN
 F 2 "~" H 2600 6350 60  0000 C CNN
@@
 	2900 6950 2900 6900
 $Comp
-L AGND #PWR066
+L AGND #PWR065
 U 1 1 54CC0292
 P 3150 7450
-F 0 "#PWR066" H 3150 7450 40  0001 C CNN
+F 0 "#PWR065" H 3150 7450 40  0001 C CNN
 F 1 "AGND" H 3150 7380 50  0000 C CNN
 F 2 "~" H 3150 7450 60  0000 C CNN
@@
 $EndComp
 $Comp
-L AGND #PWR067
+L AGND #PWR066
 U 1 1 54CC0298
 P 2900 7450
-F 0 "#PWR067" H 2900 7450 40  0001 C CNN
+F 0 "#PWR066" H 2900 7450 40  0001 C CNN
 F 1 "AGND" H 2900 7380 50  0000 C CNN
 F 2 "~" H 2900 7450 60  0000 C CNN
@@
 	1    0    0    -1
 $EndComp
+Wire Wire Line
+	4100 6000 4100 6200
+NoConn ~ 4300 6000
+$Comp
+L SW_PUSH_4PIN SW4
+U 1 1 54CE948E
+P 2600 5800
+F 0 "SW4" H 2750 5910 50  0000 C CNN
+F 1 "SW_PUSH_4PIN" H 2600 5600 50  0000 C CNN
+F 2 "~" H 2600 5800 60  0000 C CNN
+F 3 "~" H 2600 5800 60  0000 C CNN
+	1    2600 5800
+	0    -1   -1   0
+$EndComp
+$Comp
+L SW_PUSH_4PIN SW3
+U 1 1 54CE949D
+P 2200 5800
+F 0 "SW3" H 2350 5910 50  0000 C CNN
+F 1 "SW_PUSH_4PIN" H 2200 5600 50  0000 C CNN
+F 2 "~" H 2200 5800 60  0000 C CNN
+F 3 "~" H 2200 5800 60  0000 C CNN
+	1    2200 5800
+	0    -1   -1   0
+$EndComp
+Wire Wire Line
+	2200 5500 2200 5450
+Wire Wire Line
+	2200 5450 2300 5450
+Connection ~ 2300 5450
+Wire Wire Line
+	2200 6100 2200 6150
+Wire Wire Line
+	2200 6150 2300 6150
+Connection ~ 2300 6150
+Wire Wire Line
+	2600 6150 2700 6150
+Wire Wire Line
+	2700 6150 2700 6100
+Connection ~ 2600 6150
+Wire Wire Line
+	2600 5450 2700 5450
+Wire Wire Line
+	2700 5450 2700 5500
+Connection ~ 2600 5450
 $EndSCHEMATC

Commit message: Name nets for convenience on CC2540.
Connections:
- net labels added: LED1, LED2, RESET_INTR, RF_N, RF_P, SW3, SW4, USB_N_Intr, USB_P_Intr, X1_1, X1_2, X2_1, X2_3
Changed lines of the file:
@@
 	2700 5450 2700 5500
 Connection ~ 2600 5450
+Text Label 6100 4800 0    60   ~ 0
+RF_N
+Text Label 6100 4900 0    60   ~ 0
+RF_P
+Text Label 3350 6200 0    60   ~ 0
+LED2
+Text Label 2900 6000 0    60   ~ 0
+LED1
+Text Label 2550 5000 0    60   ~ 0
+SW3
+Text Label 2700 5100 0    60   ~ 0
+SW4
+Text Label 2300 4500 0    60   ~ 0
+USB_P_Intr
+Text Label 2300 4600 0    60   ~ 0
+USB_N_Intr
+Text Label 4450 3550 1    60   ~ 0
+X1_1
+Text Label 4550 3550 1    60   ~ 0
+X1_2
+Text Label 5600 5100 0    60   ~ 0
+X2_3
+Text Label 5500 5200 0    60   ~ 0
+X2_1
+Text Label 4600 6600 3    60   ~ 0
+RESET_INTR
 $EndSCHEMATC

Commit message: Continue layout for CC2540
Change swiches to one pin operating to clear under space. Edit USB conn
to show back size.
Connections:
- wire segments 118 -> 114
- no-connect marks 6 -> 8
Changed lines of the file:
@@
 Sheet 4 4
 Title "Project Synapse Prototype Board"
-Date "1 feb 2015"
+Date "2 feb 2015"
 Rev "A.b"
 Comp "Senior Design 14-15"
@@
 $EndComp
 Wire Wire Line
-	2200 5500 2200 5450
-Wire Wire Line
-	2200 5450 2300 5450
-Connection ~ 2300 5450
-Wire Wire Line
 	2200 6100 2200 6150
 Wire Wire Line
@@
 	2700 6150 2700 6100
 Connection ~ 2600 6150
-Wire Wire Line
-	2600 5450 2700 5450
-Wire Wire Line
-	2700 5450 2700 5500
-Connection ~ 2600 5450
 Text Label 6100 4800 0    60   ~ 0
 RF_N
@@
 Text Label 4600 6600 3    60   ~ 0
 RESET_INTR
+NoConn ~ 2700 5500
+NoConn ~ 2200 5500
 $EndSCHEMATC

Commit message: Continue layout, compress chips together.
Parts:
- removed X2: 32-MHz, 10/20/60/10, symbol QUARTZCMS4
- added X2: QUARTZCMS4_MOD, ~, symbol QUARTZCMS4_MOD
Changed lines of the file:
@@
 Sheet 4 4
 Title "Project Synapse Prototype Board"
-Date "2 feb 2015"
+Date "3 feb 2015"
 Rev "A.b"
 Comp "Senior Design 14-15"
@@
 F 3 "~" H 650 1400 60  0000 C CNN
 	1    650  1400
-	1    0    0    -1
-$EndComp
-$Comp
-L QUARTZCMS4 X2
-U 1 1 54B4E091
-P 6050 5750
-F 0 "X2" H 6050 5900 60  0000 C CNN
-F 1 "32-MHz" H 6050 5600 60  0000 C CNN
-F 2 "10/20/60/10" H 6050 5500 60  0000 C CNN
-F 3 "~" H 6050 5750 60  0000 C CNN
-	1    6050 5750
 	1    0    0    -1
 $EndComp
@@
 NoConn ~ 2700 5500
 NoConn ~ 2200 5500
+$Comp
+L QUARTZCMS4_MOD X2
+U 1 1 54D0201B
+P 6050 5750
+F 0 "X2" H 6050 5900 60  0000 C CNN
+F 1 "QUARTZCMS4_MOD" H 6050 5600 60  0000 C CNN
+F 2 "~" H 6050 5750 60  0000 C CNN
+F 3 "~" H 6050 5750 60  0000 C CNN
+	1    6050 5750
+	1    0    0    -1
+$EndComp
+$Comp
+L AGND #PWR067
+U 1 1 54D02032
+P 6200 5400
+F 0 "#PWR067" H 6200 5400 40  0001 C CNN
+F 1 "AGND" H 6200 5330 50  0000 C CNN
+F 2 "~" H 6200 5400 60  0000 C CNN
+F 3 "~" H 6200 5400 60  0000 C CNN
+	1    6200 5400
+	-1   0    0    1
+$EndComp
+$Comp
+L AGND #PWR068
+U 1 1 54D02038
+P 5900 5400
+F 0 "#PWR068" H 5900 5400 40  0001 C CNN
+F 1 "AGND" H 5900 5330 50  0000 C CNN
+F 2 "~" H 5900 5400 60  0000 C CNN
+F 3 "~" H 5900 5400 60  0000 C CNN
+	1    5900 5400
+	-1   0    0    1
+$EndComp
 $EndSCHEMATC

Commit message: Continue layout and add antenna
Parts:
- added A1: AN043, symbol AN043
Connections:
- wire segments 114 -> 113
Changed lines of the file:
@@
 L AGND #PWR062
 U 1 1 54C2EF06
-P 9450 4200
-F 0 "#PWR062" H 9450 4200 40  0001 C CNN
-F 1 "AGND" H 9450 4130 50  0000 C CNN
-F 2 "~" H 9450 4200 60  0000 C CNN
-F 3 "~" H 9450 4200 60  0000 C CNN
-	1    9450 4200
-	1    0    0    -1
-$EndComp
-Wire Wire Line
-	9900 4100 9900 3850
-Wire Wire Line
-	9450 3850 9450 4200
-Connection ~ 9900 3850
-Wire Wire Line
-	9450 3850 10450 3850
-Text Label 9650 3850 0    60   ~ 0
+P 9600 4100
+F 0 "#PWR062" H 9600 4100 40  0001 C CNN
+F 1 "AGND" H 9600 4030 50  0000 C CNN
+F 2 "~" H 9600 4100 60  0000 C CNN
+F 3 "~" H 9600 4100 60  0000 C CNN
+	1    9600 4100
+	1    0    0    -1
+$EndComp
+Text Label 9900 3850 0    60   ~ 0
 ANTENNA
 Text HLabel 4350 3550 1    60   Input ~ 0
@@
 	-1   0    0    1
 $EndComp
+$Comp
+L AN043 A1
+U 1 1 54D0318F
+P 9750 3300
+F 0 "A1" H 9550 3600 60  0000 C CNN
+F 1 "AN043" H 9850 3600 60  0000 C CNN
+F 2 "" H 9900 2900 60  0000 C CNN
+F 3 "" H 9900 2900 60  0000 C CNN
+	1    9750 3300
+	1    0    0    -1
+$EndComp
+Wire Wire Line
+	9900 4100 9900 3700
+Wire Wire Line
+	9600 3700 9600 4100
 $EndSCHEMATC

Commit message: Continue layout. Add fill zones.
Connections:
- net labels added: TX_LINE
Changed lines of the file:
@@
 Wire Wire Line
 	9600 3700 9600 4100
+Text Label 9900 4750 0    60   ~ 0
+TX_LINE
 $EndSCHEMATC
