File: EEG_v2.kicad_pcb (KiCad board)
At the start: 2 copper layers, 114 parts, among them P1 CONN_2, P2 CONN_8, P3 USB_A, P4 CONN_8, P5 CONN_5X2, P6 CONN_2, P7 CONN_1, SW1 SWITCH_INV, SW2 RESET, SW3 SW_PUSH_4PIN, SW4 SW_PUSH_4PIN, U1 ADS1299IPAGR, U2 TLV70033, U3 TLV70025, U4 LM2664, U5 TPS72325, U6 CC2540, U7 2450BM15A0002E, X1 QUARTZCMS4_32K, X2 QUARTZCMS4_MOD

Commit message: Continue layout and add antenna
Parts:
- added A1: AN043, AN043, F.Cu at (276.6, 145.9)
- moved R1 29.2 mm to (302.4, 168.7), turned to 270 degrees
- moved JP1 26.7 mm to (299.9, 169.4), turned to 270 degrees
- moved C56 5.80 mm to (279.5, 147.3), turned to 180 degrees
- moved R21 5.75 mm to (277.1, 147.3)
Connections:
- R21 pad 2: AGND -> /Microcontroller/ANTENNA
Routing:
- net /Analog Frontend/RESET: track 0.00 -> 20.0 mm, vias 0 -> 2
- net /Analog Frontend/DIN: track 0.00 -> 19.5 mm, vias 0 -> 2
- net /Microcontroller/SCK: track 0.00 -> 18.0 mm
- net /Analog Frontend/START: track 0.00 -> 17.8 mm
- net /Analog Frontend/CS: track 0.00 -> 17.8 mm
- net /Analog Frontend/DOUT: track 0.00 -> 17.8 mm
- net /Analog Frontend/DRDY: track 0.00 -> 17.6 mm
- net /Microcontroller/RESET_N: track 50.2 -> 58.7 mm
- net N-0000033: track 0.00 -> 3.03 mm
- net +3.3V: track 79.6 -> 81.0 mm

Commit message: Continue layout. Add fill zones.
Parts:
- moved SW1 14.8 mm to (299.0, 180.0)
- moved P7 13.7 mm to (320.0, 179.1), turned to 180 degrees
- moved P1 12.9 mm to (307.1, 179.8)
- moved R10 10.0 mm to (316.6, 178.9)
- moved R9 8.56 mm to (316.6, 177.2), turned to 180 degrees
- moved C13 8.51 mm to (316.7, 175.2), turned to 0 degrees
- moved C10 8.24 mm to (324.2, 155.9)
- moved C14 8.24 mm to (324.2, 156.9)
- moved C15 8.24 mm to (324.2, 160.3)
- moved C30 8.24 mm to (324.2, 170.2)
- moved C31 8.24 mm to (324.2, 173.7)
- moved C9 8.24 mm to (324.2, 152.5)
- moved P4 8.24 mm to (329.4, 171.0)
- moved R11 8.24 mm to (324.2, 159.2)
- moved R17 8.24 mm to (324.2, 171.4)
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Connections:
- net N-0000043 renamed /Microcontroller/TX_LINE
Routing:
- net AGND: track 143.6 -> 376.1 mm, vias 10 -> 36
- net /VBUS: track 0.00 -> 26.7 mm
- net N-0000092: track 1.18 -> 22.5 mm
- net /Analog Frontend/BIASOUT_IN: track 0.00 -> 21.1 mm
- net N-0000091: track 1.18 -> 22.2 mm
- net /Analog Frontend/BIASINV: track 0.00 -> 20.9 mm
- net N-0000096: track 1.18 -> 19.6 mm
- net N-0000095: track 1.18 -> 19.0 mm
- net VIN_RAW: track 54.5 -> 69.6 mm
- net N-0000094: track 1.18 -> 16.3 mm
- net N-0000093: track 1.18 -> 15.8 mm
- net /Analog Frontend/SRB2: track 0.00 -> 12.8 mm
- net N-00000100: track 1.18 -> 13.1 mm
- net N-0000074: track 1.18 -> 13.0 mm
- net N-0000077: track 1.18 -> 13.0 mm
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- added copper zone on B.Cu, net AGND
- added copper zone on F.Cu, net AGND
Other:
- board outline added: 66.9 x 41.5 mm
- net class TX_LINE added: clearance 0.1524, trace_width 0.35, via_dia 0.889, via_drill 0.635
- rule trace_min: 0.006 -> 0.1524
- rule via_min_size: 0.02 -> 0.508
