File: EEG_v2.kicad_pcb (KiCad board)
At the start: 2 copper layers, 66.9 x 41.5 mm, 115 parts, among them P1 CONN_2, P2 CONN_8, P3 USB_A, P4 CONN_8, P5 CONN_5X2, P6 CONN_2, P7 CONN_1, SW1 SWITCH_INV, SW2 RESET, SW3 SW_PUSH_4PIN, SW4 SW_PUSH_4PIN, U1 ADS1299IPAGR, U2 TLV70033, U3 TLV70025, U4 LM2664, U5 TPS72325, U6 CC2540, U7 2450BM15A0002E, X1 QUARTZCMS4_32K, X2 QUARTZCMS4_MOD

Commit message: Nearly finished layout
Parts:
- U6: footprint VQFN40 -> VQFN40_nodrill
Routing:
- net AGND: track 425.8 -> 667.0 mm, vias 37 -> 135
Other:
- net class Minimum: trace_width 0.1524 -> 0.254
