File: EEG_v2.sch (KiCad schematic (older format))
At the start: 11 parts, among them P1 CONN_1, P2 CONN_1, P3 CONN_8, P5 CONN_8, P6 CONN_5X2, P7 CONN_3, SW1 SWITCH_INV, SW2 RESET

Commit message: Modified Vbus on usb conn to be power out. Replaced batt connections with 0.1" headers
Parts:
- removed P1, P2: CONN_1, ~, symbol CONN_1
- added P1: CONN_2, 2x1 0.1\", symbol CONN_2
- gave numbers to parts that had none: 1
- renumbered P3 to P2, P5 to P4, P6 to P5, P7 to P6
Changed lines of the file:
@@
-$EndComp
-$Comp
-L CONN_1 P1
-U 1 1 54C44DCA
-P 1300 2800
-F 0 "P1" H 1380 2800 40  0000 L CNN
-F 1 "CONN_1" H 1300 2855 30  0001 C CNN
-F 2 "~" H 1300 2800 60  0000 C CNN
-F 3 "~" H 1300 2800 60  0000 C CNN
-	1    1300 2800
-	-1   0    0    1
-$EndComp
-$Comp
-L CONN_1 P2
-U 1 1 54C44DD9
-P 1350 3400
-F 0 "P2" H 1430 3400 40  0000 L CNN
-F 1 "CONN_1" H 1350 3455 30  0001 C CNN
-F 2 "~" H 1350 3400 60  0000 C CNN
-F 3 "~" H 1350 3400 60  0000 C CNN
-	1    1350 3400
-	-1   0    0    1
 $EndComp
 $Comp
 L AGND #PWR02
 U 1 1 54C45735
-P 1750 3500
-F 0 "#PWR02" H 1750 3500 40  0001 C CNN
-F 1 "AGND" H 1750 3430 50  0000 C CNN
-F 2 "~" H 1750 3500 60  0000 C CNN
-F 3 "~" H 1750 3500 60  0000 C CNN
-	1    1750 3500
-	1    0    0    -1
-$EndComp
-Text Label 2550 2800 0    60   ~ 0
+P 1700 3100
+F 0 "#PWR02" H 1700 3100 40  0001 C CNN
+F 1 "AGND" H 1700 3030 50  0000 C CNN
+F 2 "~" H 1700 3100 60  0000 C CNN
+F 3 "~" H 1700 3100 60  0000 C CNN
+	1    1700 3100
+	1    0    0    -1
+$EndComp
+Text Label 1500 2800 0    60   ~ 0
 BATT_+
-Text Notes 1550 3400 0    60   ~ 0
+Text Notes 1500 3000 0    60   ~ 0
 BATT_-
 $Comp
-L CONN_8 P3
+L CONN_8 P2
 U 1 1 54C84F21
 P 9100 4600
-F 0 "P3" V 9050 4600 60  0000 C CNN
+F 0 "P2" V 9050 4600 60  0000 C CNN
 F 1 "CONN_8" V 9150 4600 60  0000 C CNN
 F 2 "8x1 0.1\"" V 9300 4600 60  0000 C CNN
@@
 $EndComp
 $Comp
-L CONN_8 P5
+L CONN_8 P4
 U 1 1 54C84F2E
 P 9100 5400
-F 0 "P5" V 9050 5400 60  0000 C CNN
+F 0 "P4" V 9050 5400 60  0000 C CNN
 F 1 "CONN_8" V 9150 5400 60  0000 C CNN
 F 2 "8x1 0.1\"" V 9300 5400 60  0000 C CNN
@@
 $EndComp
 $Comp
-L CONN_3 P7
+L CONN_3 P6
 U 1 1 54C84FBA
 P 9100 5950
-F 0 "P7" V 9050 5950 50  0000 C CNN
+F 0 "P6" V 9050 5950 50  0000 C CNN
 F 1 "CONN_3" V 9150 5950 40  0000 C CNN
 F 2 "3x1 0.1\"" V 9300 5850 60  0000 C CNN
@@
 $EndComp
 $Comp
-L CONN_5X2 P6
+L CONN_5X2 P5
 U 1 1 54C8BF12
 P 2150 5700
-F 0 "P6" H 2150 6000 60  0000 C CNN
+F 0 "P5" H 2150 6000 60  0000 C CNN
 F 1 "CONN_5X2" V 2150 5700 50  0000 C CNN
 F 2 "5x2 0.1\"" H 2150 5400 60  0000 C CNN
@@
 $EndComp
 $Comp
-L USB-MINI-B CON?
+L USB-MINI-B P3
 U 1 1 54CCBB99
 P 2000 4650
-F 0 "CON?" H 1750 5100 60  0000 C CNN
+F 0 "P3" H 1750 5100 60  0000 C CNN
 F 1 "USB-MINI-B" H 1950 4150 60  0000 C CNN
 F 2 "47346-0001" H 2250 5100 60  0000 C CNN
@@
 $EndComp
 $Comp
-L AGND #PWR?
+L AGND #PWR06
 U 1 1 54CCD7A6
 P 1350 5050
-F 0 "#PWR?" H 1350 5050 40  0001 C CNN
+F 0 "#PWR06" H 1350 5050 40  0001 C CNN
 F 1 "AGND" H 1350 4980 50  0000 C CNN
 F 2 "~" H 1350 5050 60  0000 C CNN
@@
 	1450 2800 2850 2800
 Wire Wire Line
-	1500 3400 1750 3400
-Wire Wire Line
-	1750 3400 1750 3500
+	1450 3000 1700 3000
+Wire Wire Line
+	1700 3000 1700 3100
 Wire Wire Line
 	2550 5600 4900 5600
@@
 Connection ~ 1350 4800
 NoConn ~ 2550 4800
+$Comp
+L CONN_2 P1
+U 1 1 54CD8FE2
+P 1100 2900
+F 0 "P1" V 1050 2900 40  0000 C CNN
+F 1 "CONN_2" V 1150 2900 40  0000 C CNN
+F 2 "2x1 0.1\"" H 1100 3100 60  0000 C CNN
+F 3 "~" H 1100 2900 60  0000 C CNN
+	1    1100 2900
+	-1   0    0    1
+$EndComp
 $EndSCHEMATC

Commit message: Add footprints for tactile switches
Parts:
- SW2: footprint ~ -> Thru 1825910
Changed lines of the file:
@@
 F 0 "SW2" H 4750 6260 50  0000 C CNN
 F 1 "RESET" H 4600 6070 50  0000 C CNN
-F 2 "~" H 4600 6150 60  0000 C CNN
+F 2 "Thru 1825910" H 4600 6000 60  0000 C CNN
 F 3 "~" H 4600 6150 60  0000 C CNN
 	1    4600 6150
@@
 	1    4600 6550
 	1    0    0    -1
-$EndComp
-$Comp
-L USB-MINI-B P3
-U 1 1 54CCBB99
-P 2000 4650
-F 0 "P3" H 1750 5100 60  0000 C CNN
-F 1 "USB-MINI-B" H 1950 4150 60  0000 C CNN
-F 2 "47346-0001" H 2250 5100 60  0000 C CNN
-F 3 "~" H 2000 4650 60  0000 C CNN
-	1    2000 4650
-	-1   0    0    -1
 $EndComp
 $Comp
@@
 	4300 2700 4300 2900
 Wire Wire Line
-	2550 4350 2750 4350
-Wire Wire Line
 	2750 4350 2750 3000
-Wire Wire Line
-	2750 3000 2850 3000
 Wire Wire Line
 	4600 5250 4600 5850
@@
 	-1   0    0    1
 $EndComp
+Wire Wire Line
+	2750 4350 2550 4350
+Wire Wire Line
+	2750 3000 2850 3000
+$Comp
+L USB-MINI-B P3
+U 1 1 54CE6A84
+P 2000 4650
+F 0 "P3" H 1750 5100 60  0000 C CNN
+F 1 "USB-MINI-B" H 1950 4150 60  0000 C CNN
+F 2 "47346-0001" H 2150 5100 60  0000 C CNN
+F 3 "~" H 2000 4650 60  0000 C CNN
+	1    2000 4650
+	-1   0    0    -1
+$EndComp
 $EndSCHEMATC

Commit message: Add datasheet for power switch, footprints for test points
Parts:
- SW1: footprint ~ -> SSSS810701
Changed lines of the file:
@@
 F 0 "SW1" H 3150 3050 50  0000 C CNN
 F 1 "SWITCH_INV" H 3200 2750 50  0000 C CNN
-F 2 "~" H 3350 2900 60  0000 C CNN
+F 2 "SSSS810701" H 3300 3150 60  0000 C CNN
 F 3 "~" H 3350 2900 60  0000 C CNN
 	1    3350 2900

Commit message: Change USB connector. Continue layout.
Parts:
- removed P3: USB-MINI-B, 47346-0001, symbol USB-MINI-B
- removed P6: CONN_3, 3x1 0.1\", symbol CONN_3
- removed SW2: RESET, Thru 1825910, symbol SW_PUSH
- added P3: USB_A, ~, symbol USB_A
- added P6: CONN_2, 2x1 0.1\", symbol CONN_2
- added P7: CONN_1, symbol CONN_1
- added SW2: RESET, ~, symbol SW_PUSH_4PIN
Connections:
- net labels added: VBUS
- wire segments 68 -> 71
- no-connect marks 5 -> 4
Changed lines of the file:
@@
 Sheet 1 4
 Title "Project Synapse Prototype Board"
-Date "31 jan 2015"
+Date "1 feb 2015"
 Rev "A.b"
 Comp "Senior Design 14-15"
@@
 $EndComp
 $Comp
-L CONN_3 P6
-U 1 1 54C84FBA
-P 9100 5950
-F 0 "P6" V 9050 5950 50  0000 C CNN
-F 1 "CONN_3" V 9150 5950 40  0000 C CNN
-F 2 "3x1 0.1\"" V 9300 5850 60  0000 C CNN
-F 3 "~" H 9100 5950 60  0000 C CNN
-	1    9100 5950
-	1    0    0    -1
-$EndComp
-$Comp
 L CONN_5X2 P5
 U 1 1 54C8BF12
@@
 $EndComp
 $Comp
-L SW_PUSH SW2
-U 1 1 54CABD6B
-P 4600 6150
-F 0 "SW2" H 4750 6260 50  0000 C CNN
-F 1 "RESET" H 4600 6070 50  0000 C CNN
-F 2 "Thru 1825910" H 4600 6000 60  0000 C CNN
-F 3 "~" H 4600 6150 60  0000 C CNN
-	1    4600 6150
-	0    -1   -1   0
-$EndComp
-$Comp
 L AGND #PWR05
 U 1 1 54CAD291
@@
 	1    0    0    -1
 $EndComp
-$Comp
-L AGND #PWR06
-U 1 1 54CCD7A6
-P 1350 5050
-F 0 "#PWR06" H 1350 5050 40  0001 C CNN
-F 1 "AGND" H 1350 4980 50  0000 C CNN
-F 2 "~" H 1350 5050 60  0000 C CNN
-F 3 "~" H 1350 5050 60  0000 C CNN
-	1    1350 5050
-	1    0    0    -1
-$EndComp
 Wire Wire Line
 	6450 4250 7000 4250
@@
 	6450 4850 7000 4850
 Wire Wire Line
-	4900 4550 2650 4550
-Wire Wire Line
 	2550 4650 4900 4650
 Wire Wire Line
-	2550 4950 2750 4950
+	2750 4950 2550 4950
 Wire Wire Line
 	3850 2900 4900 2900
@@
 	8750 5750 8550 5750
 Wire Wire Line
-	8550 5850 8750 5850
-Wire Wire Line
-	8750 5950 8550 5950
-Wire Wire Line
-	8550 6050 8750 6050
+	8550 5850 9300 5850
+Wire Wire Line
+	8550 5950 9250 5950
+Wire Wire Line
+	8550 6050 9050 6050
 Wire Wire Line
 	1650 5550 3650 5550
@@
 	4300 2700 4300 2900
 Wire Wire Line
-	2750 4350 2750 3000
+	2750 3000 2750 4650
 Wire Wire Line
 	4600 5250 4600 5850
@@
 	4600 6450 4600 6550
 Wire Wire Line
-	2650 4550 2650 4500
-Wire Wire Line
-	2650 4500 2550 4500
-Wire Wire Line
-	2750 4950 2750 5050
-Wire Wire Line
-	1450 4950 1350 4950
-Wire Wire Line
-	1350 4350 1350 5050
-Wire Wire Line
-	1450 4350 1350 4350
-Connection ~ 1350 4950
-Wire Wire Line
-	1450 4500 1350 4500
-Connection ~ 1350 4500
-Wire Wire Line
-	1450 4800 1350 4800
-Connection ~ 1350 4800
-NoConn ~ 2550 4800
+	2750 4750 2750 5050
 $Comp
 L CONN_2 P1
@@
 $EndComp
 Wire Wire Line
-	2750 4350 2550 4350
+	2750 4650 2550 4450
+Text Label 2750 3600 1    60   ~ 0
+VBUS
+$Comp
+L USB_A P3
+U 1 1 54CDE318
+P 2250 4700
+F 0 "P3" H 2050 5200 60  0000 C CNN
+F 1 "USB_A" H 2100 5100 60  0000 C CNN
+F 2 "~" H 1800 4700 60  0000 C CNN
+F 3 "~" H 1800 4700 60  0000 C CNN
+	1    2250 4700
+	1    0    0    -1
+$EndComp
+Wire Wire Line
+	2550 4550 4900 4550
+Wire Wire Line
+	2550 4750 2750 4750
+Connection ~ 2750 4950
+Wire Wire Line
+	2550 4850 2750 4850
+Connection ~ 2750 4850
+$Comp
+L CONN_2 P6
+U 1 1 54CE5097
+P 9650 5950
+F 0 "P6" V 9600 5950 40  0000 C CNN
+F 1 "CONN_2" V 9700 5950 40  0000 C CNN
+F 2 "2x1 0.1\"" V 9850 5950 60  0000 C CNN
+F 3 "" H 9650 5950 60  0000 C CNN
+	1    9650 5950
+	1    0    0    -1
+$EndComp
+Wire Wire Line
+	9250 5950 9250 6050
+Wire Wire Line
+	9250 6050 9300 6050
+$Comp
+L CONN_1 P7
+U 1 1 54CE56CB
+P 9450 6200
+F 0 "P7" H 9530 6200 40  0000 L CNN
+F 1 "CONN_1" H 9450 6255 30  0001 C CNN
+F 2 "" H 9450 6200 60  0000 C CNN
+F 3 "" H 9450 6200 60  0000 C CNN
+	1    9450 6200
+	1    0    0    -1
+$EndComp
+Wire Wire Line
+	9050 6050 9050 6200
+Wire Wire Line
+	9050 6200 9300 6200
 Wire Wire Line
 	2750 3000 2850 3000
 $Comp
-L USB-MINI-B P3
-U 1 1 54CE6A84
-P 2000 4650
-F 0 "P3" H 1750 5100 60  0000 C CNN
-F 1 "USB-MINI-B" H 1950 4150 60  0000 C CNN
-F 2 "47346-0001" H 2150 5100 60  0000 C CNN
-F 3 "~" H 2000 4650 60  0000 C CNN
-	1    2000 4650
-	-1   0    0    -1
-$EndComp
+L SW_PUSH_4PIN SW2
+U 1 1 54CE83B3
+P 4600 6150
+F 0 "SW2" H 4750 6260 50  0000 C CNN
+F 1 "RESET" H 4600 5950 50  0000 C CNN
+F 2 "~" H 4600 6150 60  0000 C CNN
+F 3 "~" H 4600 6150 60  0000 C CNN
+	1    4600 6150
+	0    -1   -1   0
+$EndComp
+Wire Wire Line
+	4700 5850 4700 5800
+Wire Wire Line
+	4700 5800 4600 5800
+Connection ~ 4600 5800
+Wire Wire Line
+	4700 6450 4700 6500
+Wire Wire Line
+	4700 6500 4600 6500
+Connection ~ 4600 6500
 $EndSCHEMATC

Commit message: Continue layout, compress chips together.
Connections:
- wire segments 71 -> 69
- no-connect marks 4 -> 5
Changed lines of the file:
@@
 Sheet 1 4
 Title "Project Synapse Prototype Board"
-Date "2 feb 2015"
+Date "3 feb 2015"
 Rev "A.b"
 Comp "Senior Design 14-15"
@@
 $EndComp
 Wire Wire Line
-	4700 5850 4700 5800
-Wire Wire Line
-	4700 5800 4600 5800
-Connection ~ 4600 5800
-Wire Wire Line
 	4700 6450 4700 6500
 Wire Wire Line
 	4700 6500 4600 6500
 Connection ~ 4600 6500
+NoConn ~ 4700 5850
 $EndSCHEMATC

Commit message: Continue layout. Add fill zones.
Changed lines of the file:
@@
 	4300 2700 4300 2900
 Wire Wire Line
-	2750 3000 2750 4650
+	2750 3000 2750 4450
 Wire Wire Line
 	4600 5250 4600 5850
@@
 	-1   0    0    1
 $EndComp
-Wire Wire Line
-	2750 4650 2550 4450
 Text Label 2750 3600 1    60   ~ 0
 VBUS
@@
 Connection ~ 4600 6500
 NoConn ~ 4700 5850
+Wire Wire Line
+	2750 4450 2550 4450
 $EndSCHEMATC
