File: EEG_v2_auto.kicad_pcb (KiCad board)
At the start: 2 copper layers, 66.9 x 41.5 mm, 115 parts, among them P1 CONN_2, P2 CONN_8, P3 USB_A, P4 CONN_8, P5 CONN_5X2, P6 CONN_2, P7 CONN_1, SW1 SWITCH_INV, SW2 RESET, SW3 SW_PUSH_4PIN, SW4 SW_PUSH_4PIN, U1 ADS1299IPAGR, U2 TLV70033, U3 TLV70025, U4 LM2664, U5 TPS72325, U6 CC2540, U7 2450BM15A0002E, X1 QUARTZCMS4_32K, X2 QUARTZCMS4_MOD

Commit message: Tested autorouter. ehhhh.
Parts:
- removed A1: AN043, AN043
Routing:
- net /Microcontroller/VDD_FILT: track 77.0 -> 51.0 mm
- net /Microcontroller/RESET_N: track 58.7 -> 43.5 mm, vias 4 -> 1
- net +2.5V: track 42.7 -> 54.4 mm
- net /Analog Frontend/BIASOUT_IN: track 21.1 -> 28.0 mm
- net /Analog Frontend/DRDY: track 17.6 -> 23.0 mm
- net VIN_RAW: track 69.6 -> 65.2 mm
- net -2.5V: track 64.7 -> 60.9 mm
- net N-0000091: track 22.2 -> 18.5 mm
- net AGND: track 376.1 -> 379.7 mm, vias 36 -> 1
- net /Microcontroller/ANTENNA: track 3.55 -> 0.00 mm
- net N-0000095: track 19.0 -> 15.5 mm
- net N-0000093: track 15.8 -> 12.7 mm
- net N-0000096: track 19.6 -> 17.0 mm
- net N-0000092: track 22.5 -> 19.9 mm
- net /Analog Frontend/SRB2: track 12.8 -> 10.3 mm, vias 0 -> 1
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- removed copper zone on B.Cu, net AGND
- removed copper zone on F.Cu, net AGND
Other:
- rule trace_min: 0.1524 -> 0.006
- rule via_min_size: 0.508 -> 0.02
